Commit message: v3 baseline training stack: real-bench geometry, 5 any2any objects, launch + ship-gate tooling
Geometry (HANDOVER_V3 spec, tape-measured; reach audit 100% coverage):
- assets/urdf/table_real_bench.urdf (0.81x1.00 m, top at 0.184 via tableResetZ 0.034)
- env.py: tableDistanceFromBase (robot at table edge, center 0.405 m) and
  tableObjectYOffset (spawn center in the measured 0.45-0.70 m band) config
  knobs, defaults preserve v1 behavior
- franka URDF: real velocity (2.175/2.61) + effort (87/12) limits (V3 item #1)

Objects (dextoolbench/onboard_scanned_object.py, reusable for scene2/7):
- yoga_can, half_cylinder_D10_W5_scanned, salt_can, water_cup, drill_blue:
  canonical z-up meshes, CoACD decompositions, objects.py registration,
  deployment reframe jsons
- env.py objectDensityRandomization: single-object training with the paper's
  primitive mass convention (numAssetsPerType variants, density U(300,600))

Training stack:
- isaacgymenvs/launch_v3_training.py: paper SAPG config + v3 geometry, one
  GPU per run; launch_all_v3.sh starts all 6 (5 objects + primitives)
- isaacgymenvs/ship_gate_watcher.py: W&B alert + SHIP_READY marker when the
  tolerance curriculum saturates (tol 0.01, successes >= 3 sustained)
- HANDOVER_SERVER_TRAINING.md for the 8x5090 server agent

Validated locally (RTX 3070): both run types train + exit cleanly through the
launcher; density variants generate (yoga_can 87-169 g as predicted); objects
settle on the bench at correct heights across random-SO(3) spawns.

Co-Authored-By: Claude Fable 5 <noreply@anthropic.com>

File: assets/urdf/franka_right_sharpa_description/franka_right_sharpa.urdf (robot description, URDF)
Before this commit: robot franka_sharpa, 66 links, 65 joints
Joints:
- joint panda_joint1: limit lower=-2.8973001 upper=2.8973001 effort=52.1999969 velocity=10.0000005 -> lower=-2.8973001 upper=2.8973001 effort=87.0 velocity=2.175
- joint panda_joint2: limit lower=-1.7628 upper=1.7628 effort=200. velocity=10.0000005 -> lower=-1.7628 upper=1.7628 effort=87.0 velocity=2.175
- joint panda_joint3: limit lower=-2.8973001 upper=2.8973001 effort=52.1999969 velocity=10.0000005 -> lower=-2.8973001 upper=2.8973001 effort=87.0 velocity=2.175
- joint panda_joint4: limit lower=-3.0718 upper=-0.0698 effort=150. velocity=10.0000005 -> lower=-3.0718 upper=-0.0698 effort=87.0 velocity=2.175
- joint panda_joint5: limit lower=-2.8973001 upper=2.8973001 effort=7.1999998 velocity=10.0000005 -> lower=-2.8973001 upper=2.8973001 effort=12.0 velocity=2.61
- joint panda_joint6: limit lower=-0.0175 upper=3.7525 effort=7.1999998 velocity=10.0000005 -> lower=-0.0175 upper=3.7525 effort=12.0 velocity=2.61
- joint panda_joint7: limit lower=-2.8973001 upper=2.8973001 effort=7.1999998 velocity=10.0000005 -> lower=-2.8973001 upper=2.8973001 effort=12.0 velocity=2.61
